File: TAY ĐIỀU KHIỂN/TAY ĐIỀU KHIỂN.kicad_pcb (KiCad board)
At the start: 2 copper layers, 11 parts, among them U1 ESP32-WROOM-32, U2 NRF24L01_Breakout

Commit message: NEW
Parts:
- removed the ? at (139.7, 99.1)
- removed the ? at (147.3, 99.1)
- added ?: , , F.Cu at (96.5, 101.6)
- added ?: , , F.Cu at (147.3, 101.6)
- C4: value 100uF -> C
- U1: value ESP32-WROOM-32 -> ESP32-DevKitC; footprint Connector_PinHeader_2.54mm:PinHeader_2x19_P2.54mm_Vertical -> PCM_Espressif:ESP32-DevKitC
- moved litium 96.7 mm to (167.6, 61.0), turned to 180 degrees
- moved C4 89.8 mm to (162.6, 58.4), turned to -90 degrees
- moved U1 23.0 mm to (99.1, 127.0)
- moved C3 5.68 mm to (116.8, 61.0)
- moved U2 5.68 mm to (121.9, 63.5)
- moved C1 2.50 mm to (106.7, 81.3), turned to -90 degrees
Connections:
- C1 pad 1: (no net) -> +3.3V
- C1 pad 2: (no net) -> GND
- C2 pad 1: (no net) -> GND
- C2 pad 2: (no net) -> +3.3V
- C3 pad 2: Net-(JoystickPS2-1-VCC) -> GND
- C4 pad 1: (no net) -> Net-(C4-Pad1)
- C4 pad 2: (no net) -> Net-(U1-5V)
- JoystickPS2-1 pad 3: unconnected-(U1-IO13-Pad16) -> (no net)
- JoystickPS2-1 pad 4: unconnected-(U1-IO12-Pad14) -> (no net)
- JoystickPS2-1 pad 5: unconnected-(U1-IO14-Pad13) -> (no net)
- JoystickPS2-2 pad 4: unconnected-(U1-IO34-Pad6) -> (no net)
- JoystickPS2-2 pad 5: unconnected-(U1-IO35-Pad7) -> (no net)
- U1 pad 1: +1V0 -> unconnected-(U1-3V3-Pad1)
- U1 pad 10: unconnected-(U1-IO13-Pad16) -> unconnected-(U1-DAC_2/ADC2_CH9/GPIO26-Pad10)
- U1 pad 11: unconnected-(U1-IO26-Pad11) -> unconnected-(U1-ADC2_CH7/GPIO27-Pad11)
- U1 pad 12: Net-(JoystickPS2-1-VCC) -> unconnected-(U1-MTMS/GPIO14/ADC2_CH6-Pad12)
- U1 pad 13: unconnected-(U1-IO14-Pad13) -> unconnected-(U1-MTDI/GPIO12/ADC2_CH5-Pad13)
- U1 pad 14: unconnected-(U1-IO12-Pad14) -> Net-(C4-Pad1)
- U1 pad 15: +1V0 -> unconnected-(U1-MTCK/GPIO13/ADC2_CH4-Pad15)
- U1 pad 16: unconnected-(U1-IO14-Pad13) -> unconnected-(U1-SD_DATA2/GPIO9-Pad16)
- U1 pad 17: unconnected-(U1-SHD/SD2-Pad17) -> unconnected-(U1-SD_DATA3/GPIO10-Pad17)
- U1 pad 18: unconnected-(U1-IO27-Pad12) -> unconnected-(U1-CMD-Pad18)
- U1 pad 19: unconnected-(U1-SCS/CMD-Pad19) -> Net-(U1-5V)
- U1 pad 2: Net-(U1-VDD) -> unconnected-(U1-CHIP_PU-Pad2)
- U1 pad 20: unconnected-(U1-IO26-Pad11) -> unconnected-(U1-SD_CLK/GPIO6-Pad20)
- U1 pad 22: unconnected-(U1-IO25-Pad10) -> unconnected-(U1-SD_DATA1/GPIO8-Pad22)
- U1 pad 24: unconnected-(U1-IO33-Pad9) -> unconnected-(U1-ADC2_CH2/GPIO2-Pad24)
- U1 pad 25: unconnected-(U1-IO0-Pad25) -> VR - Y2
- U1 pad 26: unconnected-(U1-IO32-Pad8) -> VR - X1
- U1 pad 28: unconnected-(U1-IO35-Pad7) -> CE
- U1 pad 29: unconnected-(U1-IO5-Pad29) -> CSN
- U1 pad 3: unconnected-(U1-EN-Pad3) -> unconnected-(U1-SENSOR_VP/GPIO36/ADC1_CH0-Pad3)
- U1 pad 30: unconnected-(U1-IO34-Pad6) -> SCK
- U1 pad 31: unconnected-(U1-IO19-Pad31) -> MISO
- U1 pad 32: unconnected-(U1-NC-Pad32) -> Net-(C4-Pad1)
- U1 pad 33: unconnected-(U1-IO21-Pad33) -> SW2
- U1 pad 34: unconnected-(U1-SWP/SD3-Pad18) -> unconnected-(U1-U0RXD/GPIO3-Pad34)
- U1 pad 36: unconnected-(U1-EN-Pad3) -> SW1
- U1 pad 37: unconnected-(U1-IO23-Pad37) -> MOSI
- U1 pad 38: +3.3V -> Net-(C4-Pad1)
- U1 pad 4: unconnected-(U1-SCS/CMD-Pad19) -> unconnected-(U1-SENSOR_VN/GPIO39/ADC1_CH3-Pad4)
- U1 pad 6: unconnected-(U1-SWP/SD3-Pad18) -> unconnected-(U1-VDET_2/GPIO35/ADC1_CH7-Pad6)
- U1 pad 7: unconnected-(U1-IO35-Pad7) -> unconnected-(U1-32K_XP/GPIO32/ADC1_CH4-Pad7)
- U1 pad 8: unconnected-(U1-SHD/SD2-Pad17) -> unconnected-(U1-32K_XN/GPIO33/ADC1_CH5-Pad8)
- U1 pad 9: unconnected-(U1-IO33-Pad9) -> unconnected-(U1-DAC_1/ADC2_CH8/GPIO25-Pad9)
- U2 pad 1: Net-(JoystickPS2-1-VCC) -> GND
- U2 pad 3: unconnected-(U1-IO26-Pad11) -> CE
- U2 pad 4: unconnected-(U1-IO27-Pad12) -> CSN
- U2 pad 5: unconnected-(U1-IO25-Pad10) -> SCK
- U2 pad 6: unconnected-(U1-IO32-Pad8) -> MOSI
- U2 pad 7: unconnected-(U1-IO33-Pad9) -> MISO
- litium pad 1: (no net) -> +3.3V
- litium pad 2: (no net) -> GND
Routing:
- net unconnected-(U1-3V3-Pad1): track 0.00 -> 183.0 mm, vias 0 -> 7
- net (no net): track 177.6 -> 0.00 mm, vias 5 -> 0
- net GND: track 0.00 -> 172.4 mm, vias 0 -> 4
- net Net-(JoystickPS2-1-VCC): track 149.0 -> 0.00 mm, vias 7 -> 0
- net +3.3V: track 113.8 -> 10.3 mm, vias 5 -> 0
- net Net-(U1-5V): track 0.00 -> 93.3 mm, vias 0 -> 2
- net MOSI: track 0.00 -> 76.2 mm, vias 0 -> 4
- net CSN: track 0.00 -> 63.5 mm
- net unconnected-(U1-IO27-Pad12): track 63.1 -> 0.00 mm
- net unconnected-(U1-IO32-Pad8): track 56.9 -> 0.00 mm
- net MISO: track 0.00 -> 50.8 mm, vias 0 -> 2
- net SCK: track 0.00 -> 45.7 mm, vias 0 -> 2
- net unconnected-(U1-IO33-Pad9): track 42.7 -> 0.00 mm
- net unconnected-(U1-IO25-Pad10): track 42.7 -> 0.00 mm
- net unconnected-(U1-IO26-Pad11): track 42.7 -> 0.00 mm
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Other:
- board text added: "3V3"
- board text added: "5V"
